File: Hardware/MeshProto.sch (KiCad schematic (older format))
At the start: 23 parts, among them P1 CONN_1, P10 CONN_1, P11 CONN_1, P12 CONN_1, P13 CONN_1, P14 CONN_1, P15 CONN_1, P16 CONN_1, P17 CONN_1, P18 CONN_1, P19 CONN_1, P2 CONN_1, P20 CONN_1, P3 CONN_1, P4 CONN_1, P5 CONN_1, P6 CONN_1, P7 CONN_1, P8 CONN_1, P9 CONN_1, U1 XBEE

Commit message: v02
Parts:
- added P21, P22, P23, P24, P25, P26, P27, P28, P29, P30, P31, P32, P33, P34, P35, P36, P37, P38, P39, P40, P41, P42, P43, P44, P45, P46, P47, P48, P49, P50, P51, P52, P53, P54, P55, P56, P57, P58, P59, P60, P61, P62, P63, P64, P65, P66, P67, P68, P69, P70, P71, P72, P73, P74, P75, P76, P77, P78, P79, P80: CONN_1, symbol CONN_1
Connections:
- no-connect marks 20 -> 80
Other:
- moved on the sheet: H1, H2, P1, P10, P11, P12, P13, P14, P15, P16, P17, P18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

Commit message: Layout Almost Complete
Parts:
- added P81, P82, P83, P84, P85, P86, P87, P88, P89, P90, P91, P92, P93, P94: CONN_1, symbol CONN_1
- added SW1: SPST, ~, symbol SPST
- H1, H2: footprint (none) -> _MP_XbeeTH10Pin
- P1, P10, P11, P12, P13, P14, P15, P16, P17, P18, P19, P2, P20, P3, P4, P5, P6, P7, P8, P9: footprint (none) -> PIN_ARRAY_1
- P21, P22, P23, P24, P25, P26, P27, P28, P29, P30, P31, P32, P33, P34, P35, P36, P37, P38, P39, P40, P41, P42, P43, P44, P45, P46, P47, P48, P49, P50, P51, P52, P53, P54, P55, P56, P57, P58, P59, P60, P61, P62, P63, P64, P65, P66, P67, P68, P69, P70, P71, P72, P73, P74, P75, P76, P77, P78, P79, P80: footprint (none) -> _MP_1Pin
- U1: footprint (none) -> _MUSB_XBee_Board_OUTLINE_ONLY
Connections:
- wire segments 23 -> 29

Commit message: Initial changes to v1.2.
Parts:
- removed SW1: SPST, ~, symbol SPST
- added P100, P101, P102, P103, P104, P105, P106, P107, P108, P95, P96, P97, P98, P99: CONN_1, _MP_1Pin, symbol CONN_1
Connections:
- wire segments 29 -> 23
- no-connect marks 80 -> 94
Changed lines of the file:
@@
 LIBS:contrib
 LIBS:valves
-LIBS:MeshProto
-LIBS:modules_droids
-LIBS:MeshThing-cache
+LIBS:MeshThing
+LIBS:MeshUSB
 LIBS:MeshProto-cache
-EELAYER 27 0
+EELAYER 24 0
 EELAYER END
 $Descr A4 11693 8268
@@
 Sheet 1 1
 Title "MeshProto by Robert Powers & David Chanter"
-Date "12 nov 2013"
-Rev "v0.1"
+Date "27 Feb 2014"
+Rev "v1.2"
 Comp "MeshAge"
 Comment1 ""
@@
 Wire Wire Line
 	5950 3400 6100 3400
-Wire Wire Line
-	2100 3550 2400 3550
-$Comp
-L SPST SW1
-U 1 1 528212C5
-P 1200 3650
-F 0 "SW1" H 1200 3750 70  0000 C CNN
-F 1 "SPST" H 1200 3550 70  0000 C CNN
-F 2 "~" H 1200 3650 60  0000 C CNN
-F 3 "~" H 1200 3650 60  0000 C CNN
-	1    1200 3650
-	1    0    0    -1
-$EndComp
-Wire Wire Line
-	1700 3650 2100 3650
-Wire Wire Line
-	2100 3650 2100 3550
-Wire Wire Line
-	700  3650 700  2950
-Wire Wire Line
-	700  2950 2300 2950
-Wire Wire Line
-	2300 2950 2300 2900
 Connection ~ 2300 2900
 $Comp
@@
 Connection ~ 2400 3950
 Connection ~ 2400 4050
+$Comp
+L CONN_1 P99
+U 1 1 530EB91E
+P 7250 4400
+F 0 "P99" H 7330 4400 40  0000 L CNN
+F 1 "CONN_1" H 7250 4455 30  0001 C CNN
+F 2 "_MP_1Pin" H 7250 4400 60  0000 C CNN
+F 3 "" H 7250 4400 60  0000 C CNN
+	1    7250 4400
+	-1   0    0    1
+$EndComp
+$Comp
+L CONN_1 P100
+U 1 1 530EB924
+P 7250 4500
+F 0 "P100" H 7330 4500 40  0000 L CNN
+F 1 "CONN_1" H 7250 4555 30  0001 C CNN
+F 2 "_MP_1Pin" H 7250 4500 60  0000 C CNN
+F 3 "" H 7250 4500 60  0000 C CNN
+	1    7250 4500
+	-1   0    0    1
+$EndComp
+$Comp
+L CONN_1 P101
+U 1 1 530EB92A
+P 7250 4600
+F 0 "P101" H 7330 4600 40  0000 L CNN
+F 1 "CONN_1" H 7250 4655 30  0001 C CNN
+F 2 "_MP_1Pin" H 7250 4600 60  0000 C CNN
+F 3 "" H 7250 4600 60  0000 C CNN
+	1    7250 4600
+	-1   0    0    1
+$EndComp
+$Comp
+L CONN_1 P102
+U 1 1 530EB930
+P 7250 4700
+F 0 "P102" H 7330 4700 40  0000 L CNN
+F 1 "CONN_1" H 7250 4755 30  0001 C CNN
+F 2 "_MP_1Pin" H 7250 4700 60  0000 C CNN
+F 3 "" H 7250 4700 60  0000 C CNN
+	1    7250 4700
+	-1   0    0    1
+$EndComp
+$Comp
+L CONN_1 P103
+U 1 1 530EB936
+P 7250 4800
+F 0 "P103" H 7330 4800 40  0000 L CNN
+F 1 "CONN_1" H 7250 4855 30  0001 C CNN
+F 2 "_MP_1Pin" H 7250 4800 60  0000 C CNN
+F 3 "" H 7250 4800 60  0000 C CNN
+	1    7250 4800
+	-1   0    0    1
+$EndComp
+$Comp
+L CONN_1 P104
+U 1 1 530EB93C
+P 7250 4900
+F 0 "P104" H 7330 4900 40  0000 L CNN
+F 1 "CONN_1" H 7250 4955 30  0001 C CNN
+F 2 "_MP_1Pin" H 7250 4900 60  0000 C CNN
+F 3 "" H 7250 4900 60  0000 C CNN
+	1    7250 4900
+	-1   0    0    1
+$EndComp
+$Comp
+L CONN_1 P105
+U 1 1 530EB942
+P 7250 5000
+F 0 "P105" H 7330 5000 40  0000 L CNN
+F 1 "CONN_1" H 7250 5055 30  0001 C CNN
+F 2 "_MP_1Pin" H 7250 5000 60  0000 C CNN
+F 3 "" H 7250 5000 60  0000 C CNN
+	1    7250 5000
+	-1   0    0    1
+$EndComp
+$Comp
+L CONN_1 P106
+U 1 1 530EB948
+P 7250 5100
+F 0 "P106" H 7330 5100 40  0000 L CNN
+F 1 "CONN_1" H 7250 5155 30  0001 C CNN
+F 2 "_MP_1Pin" H 7250 5100 60  0000 C CNN
+F 3 "" H 7250 5100 60  0000 C CNN
+	1    7250 5100
+	-1   0    0    1
+$EndComp
+$Comp
+L CONN_1 P107
+U 1 1 530EB94E
+P 7250 5200
+F 0 "P107" H 7330 5200 40  0000 L CNN
+F 1 "CONN_1" H 7250 5255 30  0001 C CNN
+F 2 "_MP_1Pin" H 7250 5200 60  0000 C CNN
+F 3 "" H 7250 5200 60  0000 C CNN
+	1    7250 5200
+	-1   0    0    1
+$EndComp
+$Comp
+L CONN_1 P108
+U 1 1 530EB954
+P 7250 5300
+F 0 "P108" H 7330 5300 40  0000 L CNN
+F 1 "CONN_1" H 7250 5355 30  0001 C CNN
+F 2 "_MP_1Pin" H 7250 5300 60  0000 C CNN
+F 3 "" H 7250 5300 60  0000 C CNN
+	1    7250 5300
+	-1   0    0    1
+$EndComp
+$Comp
+L CONN_1 P95
+U 1 1 530EB95A
+P 6700 4400
+F 0 "P95" H 6780 4400 40  0000 L CNN
+F 1 "CONN_1" H 6700 4455 30  0001 C CNN
+F 2 "_MP_1Pin" H 6700 4400 60  0000 C CNN
+F 3 "" H 6700 4400 60  0000 C CNN
+	1    6700 4400
+	-1   0    0    1
+$EndComp
+$Comp
+L CONN_1 P96
+U 1 1 530EB960
+P 6700 4500
+F 0 "P96" H 6780 4500 40  0000 L CNN
+F 1 "CONN_1" H 6700 4555 30  0001 C CNN
+F 2 "_MP_1Pin" H 6700 4500 60  0000 C CNN
+F 3 "" H 6700 4500 60  0000 C CNN
+	1    6700 4500
+	-1   0    0    1
+$EndComp
+$Comp
+L CONN_1 P97
+U 1 1 530EB966
+P 6700 4600
+F 0 "P97" H 6780 4600 40  0000 L CNN
+F 1 "CONN_1" H 6700 4655 30  0001 C CNN
+F 2 "_MP_1Pin" H 6700 4600 60  0000 C CNN
+F 3 "" H 6700 4600 60  0000 C CNN
+	1    6700 4600
+	-1   0    0    1
+$EndComp
+$Comp
+L CONN_1 P98
+U 1 1 530EB96C
+P 6700 4700
+F 0 "P98" H 6780 4700 40  0000 L CNN
+F 1 "CONN_1" H 6700 4755 30  0001 C CNN
+F 2 "_MP_1Pin" H 6700 4700 60  0000 C CNN
+F 3 "" H 6700 4700 60  0000 C CNN
+	1    6700 4700
+	-1   0    0    1
+$EndComp
+NoConn ~ 6850 4400
+NoConn ~ 6850 4500
+NoConn ~ 6850 4600
+NoConn ~ 6850 4700
+NoConn ~ 7400 4400
+NoConn ~ 7400 4500
+NoConn ~ 7400 4600
+NoConn ~ 7400 4700
+NoConn ~ 7400 4800
+NoConn ~ 7400 4900
+NoConn ~ 7400 5000
+NoConn ~ 7400 5100
+NoConn ~ 7400 5200
+NoConn ~ 7400 5300
 $EndSCHEMATC
